File: canbus.kicad_sch (KiCad schematic)
At the start: 3 parts, among them U4 MCP2518FD-xQBB, U5 ISO1044BD

Commit message: m2003 drive
Parts:
- removed PS1: MIE1W0505BGLVH-3R-Z, MSic:CONV_MIE1W0505BGLVH-3R-Z, symbol MSic:MIE1W0505BGLVH-3R-Z
- added PS2: MIE1W0505BGLVH-3R-Z, PMIC:CONV_MIE1W0505BGLVH-3R-Z, symbol PMIC-regulator:MIE1W0505BGLVH-3R-Z
Changed lines of the file:
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@@
 	)
 	(symbol
-		(lib_id "MSic:MIE1W0505BGLVH-3R-Z")
-		(at 121.92 125.73 0)
+		(lib_id "PMIC-regulator:MIE1W0505BGLVH-3R-Z")
+		(at 123.19 121.285 0)
 		(unit 1)
 		(body_style 1)
@@
 		(dnp no)
 		(fields_autoplaced yes)
-		(property "Reference" "PS1"
-			(at 121.92 110.49 0)
+		(property "Reference" "PS2"
+			(at 123.19 106.045 0)
 			(show_name no)
 			(do_not_autoplace no)
@@
 		)
 		(property "Value" "MIE1W0505BGLVH-3R-Z"
-			(at 121.92 113.03 0)
+			(at 123.19 108.585 0)
 			(show_name no)
 			(do_not_autoplace no)
@@
 			)
 		)
-		(property "Footprint" "MSic:CONV_MIE1W0505BGLVH-3R-Z"
-			(at 121.92 125.73 0)
+		(property "Footprint" "PMIC:CONV_MIE1W0505BGLVH-3R-Z"
+			(at 123.19 121.285 0)
 			(hide yes)
 			(show_name no)
@@
 		)
 		(property "Datasheet" ""
-			(at 121.92 125.73 0)
+			(at 123.19 121.285 0)
 			(hide yes)
 			(show_name no)
@@
 		)
 		(property "Description" ""
-			(at 121.92 125.73 0)
+			(at 123.19 121.285 0)
 			(hide yes)
 			(show_name no)
@@
 		)
 		(property "PARTREV" "0.8"
-			(at 121.92 125.73 0)
+			(at 123.19 121.285 0)
 			(hide yes)
 			(show_name no)
@@
 		)
 		(property "STANDARD" "Manufacturer Recommendations"
-			(at 121.92 125.73 0)
+			(at 123.19 121.285 0)
 			(hide yes)
 			(show_name no)
@@
 		)
 		(property "MAXIMUM_PACKAGE_HEIGHT" "1.28mm"
-			(at 121.92 125.73 0)
+			(at 123.19 121.285 0)
 			(hide yes)
 			(show_name no)
@@
 		)
 		(property "MANUFACTURER" "Monolithic Power Systems Inc."
-			(at 121.92 125.73 0)
+			(at 123.19 121.285 0)
 			(hide yes)
 			(show_name no)
@@
 			)
 		)
+		(pin "5_6"
+		)
 		(pin "9_10"
 		)
+		(pin "3_4"
+		)
+		(pin "8"
+		)
+		(pin "7"
+		)
 		(pin "1"
-		)
-		(pin "5_6"
 		)
 		(pin "11_12"
@@
 		(pin "2"
 		)
-		(pin "7"
-		)
-		(pin "8"
-		)
-		(pin "3_4"
-		)
 		(instances
 			(project "drive"
 				(path "/8fcb549a-cfcf-410d-b0cb-2819149beb55/f291c1ee-6428-4bfa-b73e-99eb2a9dba27"
-					(reference "PS1")
+					(reference "PS2")
 					(unit 1)
 				)
