File: microcontroller.kicad_sch (KiCad schematic)
At the start: 43 parts, among them J13 USB_C_Receptacle_USB2.0_16P, J15 USB_C_Receptacle_USB2.0_16P, Q1 DMG1012T, SW1 PTS810SJG250SMTRLFS, SW2 PTS810SJG250SMTRLFS, U2 RP2350A, U3 W25Q128JVPIQ, X1 ABM8-272-T3

Commit message: m2003 drive
Parts:
- removed C19: 0.1uF, Capacitor_SMD:C_0402_1005Metric, symbol kuleana:C
- removed J13, J15: USB_C_Receptacle_USB2.0_16P, MSconnector:USB_C_Receptacle_GCT_USB4115-03-C, symbol kuleana:USB_C_Receptacle_USB2.0_16P
- removed R19: 1k, Resistor_SMD:R_0402_1005Metric, symbol kuleana:R
- removed R20: 1M, Resistor_SMD:R_0402_1005Metric, symbol kuleana:R
- added J1: USB_C_Receptacle, Connector_USB:USB_C_Receptacle_GCT_USB4115-03-C, symbol Connector:USB_C_Receptacle
- U2: footprint Package_DFN_QFN:QFN-60-1EP_7x7mm_P0.4mm_EP3.4x3.4mm -> MCU:RP2350-QFN-60-1EP_7x7_P0.4mm_EP3.4x3.4mm_ThermalVias
Connections:
- net CC1: now also J1.A5 (CC1); no longer U2.40 (GPIO26/ADC0)
- net CC2: now also J1.B5 (CC2); no longer U2.41 (GPIO27/ADC1)
- net GND: now also J1.A1 (GND), J1.A12 (GND), J1.B1 (GND), J1.B12 (GND), J1.SH (SHIELD)
- net USB_D_N: now also J1.A7 (D-), J1.B7 (D-)
- net USB_D_P: now also J1.A6 (D+), J1.B6 (D+)
- net VBUS: now also J1.A4 (VBUS), J1.A9 (VBUS), J1.B4 (VBUS), J1.B9 (VBUS)
- net INLC: now reaches U2.10 (GPIO7)
- net SPI1_SCK: now reaches U2.14 (GPIO10)
- net SPI1_MOSI: now reaches U2.15 (GPIO11)
- net SPI1_MISO: now reaches U2.16 (GPIO12)
- net CAN_CS: now reaches U2.17 (GPIO13)
- net ENC_CS: now reaches U2.18 (GPIO14)
- net VREF/ILIM: now reaches U2.19 (GPIO15)
- net SPI0_MISO: now reaches U2.27 (GPIO16)
- net DRV_CS: now reaches U2.28 (GPIO17)
- net SPI0_SCK: now reaches U2.29 (GPIO18)
- net SPI0_MOSI: now reaches U2.31 (GPIO19)
- net DRV_FAULT: now reaches U2.32 (GPIO20)
- net DRV_OFF: now reaches U2.33 (GPIO21)
- net INHA: now reaches U2.4 (GPIO2)
- net INLA: now reaches U2.5 (GPIO3)
- net INHB: now reaches U2.7 (GPIO4)
- net INLB: now reaches U2.8 (GPIO5)
- net INHC: now reaches U2.9 (GPIO6)
- net 1V1_ADC renamed DRV_CSC
- new net DRV_CSA: U2.40 (GPIO26/ADC0)
- new net DRV_CSB: U2.41 (GPIO27/ADC1)
- no-connect marks 8 -> 14
Other:
- moved on the sheet: D1, D2, R5, R6
