File: drive.kicad_pcb (KiCad board)
At the start: 2 copper layers, 48 x 48 mm, 61 parts, among them J13 USB_C_Receptacle_USB2.0_16P, J14 FTSH-105-01-L-DV-K-P, J15 USB_C_Receptacle_USB2.0_16P, Q1 DMG1012T, SW1 PTS810SJG250SMTRLFS, SW2 PTS810SJG250SMTRLFS, U1 DRV8316RRGFR, U2 RP2350A, U3 W25Q128JVPIQ, U4 MCP2518FD-xQBB, U5 ISO1044BD, X1 ABM8-272-T3

Commit message: m2003 drive
Parts:
- removed C19: 0.1uF, Capacitor_SMD:C_0402_1005Metric
- removed J13, J15: USB_C_Receptacle_USB2.0_16P, MSconnector:USB_C_Receptacle_GCT_USB4115-03-C
- removed J14: FTSH-105-01-L-DV-K-P, kuleana:SAMTEC_FTSH-105-XX-X-DV
- removed PS1: MIE1W0505BGLVH-3R-Z, MSic:CONV_MIE1W0505BGLVH-3R-Z
- removed R19: 1k, Resistor_SMD:R_0402_1005Metric
- removed R20: 1M, Resistor_SMD:R_0402_1005Metric
- added C28: 47uF, Capacitor_SMD:C_0805_2012Metric, F.Cu at (156.9, 72.2)
- added C29: 47uF, Capacitor_SMD:C_0805_2012Metric, F.Cu at (156.9, 75.2)
- added J1: USB_C_Receptacle, Connector_USB:USB_C_Receptacle_GCT_USB4115-03-C, F.Cu at (143.0, 79.4)
- added J2: ~, xt30:XT30(2+2)PB-M.G.B, F.Cu at (129.6, 85.8)
- added J3: ~, xt30:XT30(2+2)PB-M.G.B, F.Cu at (135.2, 85.8)
- added PS2: MIE1W0505BGLVH-3R-Z, PMIC:CONV_MIE1W0505BGLVH-3R-Z, F.Cu at (174.0, 80.6)
- SW2: moved to B.Cu
- U1: footprint MSic:RGF0040E-MFG -> DRV8316:drv
- U2: footprint Package_DFN_QFN:QFN-60-1EP_7x7mm_P0.4mm_EP3.4x3.4mm -> MCU:RP2350-QFN-60-1EP_7x7_P0.4mm_EP3.4x3.4mm_ThermalVias
- moved R9 62.8 mm to (138.2, 73.2)
- moved R8 61.0 mm to (143.0, 73.4)
- moved R15 60.5 mm to (146.6, 74.0)
- moved U4 56.6 mm to (180.4, 72.8)
- moved U5 56.6 mm to (170.0, 67.8)
- moved R22 52.1 mm to (165.0, 87.2)
- moved X1 40.0 mm to (162.6, 103.8), turned to -90 degrees
- moved C26 36.6 mm to (136.4, 113.0), turned to -30 degrees
- moved U2 34.5 mm to (168.9, 102.9)
- moved D1 33.7 mm to (150.0, 77.5)
- moved D2 33.7 mm to (150.0, 81.5)
- moved U1 33.6 mm to (141.4, 115.6), turned to 60 degrees
- moved TP1 23.4 mm to (154.2, 121.2)
- moved U3 22.3 mm to (167.7, 94.2)
- moved C10 20.1 mm to (145.8, 119.0)
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Connections:
- C2 pad 1: Net-(C2-Pad1) -> VBUS
- C22 pad 1: Net-(C2-Pad1) -> VBUS
- C23 pad 1: Net-(C2-Pad1) -> VBUS
- C24 pad 1: Net-(C2-Pad1) -> VBUS
- C25 pad 1: Net-(C2-Pad1) -> VBUS
- U1 pad 10: Net-(C2-Pad1) -> VBUS
- U1 pad 11: Net-(C2-Pad1) -> VBUS
- U1 pad 9: Net-(C2-Pad1) -> VBUS
- U2 pad 10: unconnected-(U2-GPIO7-Pad10) -> /microcontroller/INLC
- U2 pad 14: unconnected-(U2-GPIO10-Pad14) -> /microcontroller/SPI1_SCK
- U2 pad 15: unconnected-(U2-GPIO11-Pad15) -> /microcontroller/SPI1_MOSI
- U2 pad 16: unconnected-(U2-GPIO12-Pad16) -> /microcontroller/SPI1_MISO
- U2 pad 17: unconnected-(U2-GPIO13-Pad17) -> /microcontroller/CAN_CS
- U2 pad 18: unconnected-(U2-GPIO14-Pad18) -> /microcontroller/ENC_CS
- U2 pad 19: unconnected-(U2-GPIO15-Pad19) -> /microcontroller/VREF/ILIM
- U2 pad 27: unconnected-(U2-GPIO16-Pad27) -> /microcontroller/SPI0_MISO
- U2 pad 28: unconnected-(U2-GPIO17-Pad28) -> /microcontroller/DRV_CS
- U2 pad 29: unconnected-(U2-GPIO18-Pad29) -> /microcontroller/SPI0_SCK
- U2 pad 31: unconnected-(U2-GPIO19-Pad31) -> /microcontroller/SPI0_MOSI
- U2 pad 32: unconnected-(U2-GPIO20-Pad32) -> /microcontroller/DRV_FAULT
- U2 pad 33: unconnected-(U2-GPIO21-Pad33) -> /microcontroller/DRV_OFF
- U2 pad 4: unconnected-(U2-GPIO2-Pad4) -> /microcontroller/INHA
- U2 pad 40: /microcontroller/CC1 -> /microcontroller/DRV_CSA
- U2 pad 41: /microcontroller/CC2 -> /microcontroller/DRV_CSB
- U2 pad 42: /microcontroller/1V1_ADC -> /microcontroller/DRV_CSC
- U2 pad 5: unconnected-(U2-GPIO3-Pad5) -> /microcontroller/INLA
- U2 pad 7: unconnected-(U2-GPIO4-Pad7) -> /microcontroller/INHB
- U2 pad 8: unconnected-(U2-GPIO5-Pad8) -> /microcontroller/INLB
- U2 pad 9: unconnected-(U2-GPIO6-Pad9) -> /microcontroller/INHC

Commit message: schematic complete
Parts:
- removed C10, C12, C13, C16, C18, C5, C6, C7, C9: 100n, Capacitor_SMD:C_0402_1005Metric
- removed C11, C14, C15, C17: 4.7u, Capacitor_SMD:C_0402_1005Metric
- removed C20: 0.1uF, Capacitor_SMD:C_0402_1005Metric
- removed C21: 1uF, Capacitor_SMD:C_0402_1005Metric
- removed C22, C23, C24, C25, C28, C29: 47uF, Capacitor_SMD:C_0805_2012Metric
- removed C26: 100nF, Capacitor_SMD:C_0402_1005Metric
- removed C27: 22uF, Capacitor_SMD:C_0805_2012Metric
- removed C3: 10uF, Capacitor_SMD:C_0402_1005Metric
- removed C4, C8: 15pF, Capacitor_SMD:C_0402_1005Metric
- removed D1: Orange, LED_SMD:LED_0603_1608Metric
- removed D2: Green, LED_SMD:LED_0603_1608Metric
- removed J1: USB_C_Receptacle, Connector_USB:USB_C_Receptacle_GCT_USB4115-03-C
- removed J3: ~, xt30:XT30(2+2)PB-M.G.B
- removed PS2: MIE1W0505BGLVH-3R-Z, PMIC:CONV_MIE1W0505BGLVH-3R-Z
- removed Q1: DMG1012T, Package_TO_SOT_SMD:SOT-523
- removed R10, R9: 27.4, Resistor_SMD:R_0402_1005Metric
- removed R11: 33, Resistor_SMD:R_0402_1005Metric
- removed R12, R22: 1k, Resistor_SMD:R_0402_1005Metric
- removed R16: 100k, Resistor_SMD:R_0402_1005Metric
- removed R21: dnf, Resistor_SMD:R_0402_1005Metric
- removed R7, R8: 5.1k, Resistor_SMD:R_0402_1005Metric
- removed SW1, SW2: PTS810SJG250SMTRLFS, Button_Switch_SMD:SW_SPST_PTS810
- removed TP1: Motor_A, TestPoint:TestPoint_Plated_Hole_D2.0mm
- removed TP2: Motor_B, TestPoint:TestPoint_Plated_Hole_D2.0mm
- removed TP3: Motor_C, TestPoint:TestPoint_Plated_Hole_D2.0mm
- removed U5: ISO1044BD, Package_SO:SOIC-8_3.9x4.9mm_P1.27mm
- removed X1: ABM8-272-T3, Crystal:Crystal_SMD_Abracon_ABM8G-4Pin_3.2x2.5mm
- added C19: 1nF, Capacitor_SMD:C_0402_1005Metric, F.Cu at (182.8, 78.3)
- added C30: 1nF, Capacitor_SMD:C_0402_1005Metric, F.Cu at (182.8, 80.3)
- added C31: 1nF, Capacitor_SMD:C_0402_1005Metric, F.Cu at (182.8, 82.3)
- added C32: 0.1uF, Capacitor_SMD:C_0402_1005Metric, F.Cu at (182.8, 84.2)
- added C33: 0.1uF, Capacitor_SMD:C_0402_1005Metric, F.Cu at (186.8, 73.8)
- added C34: 22uF, Capacitor_SMD:C_0805_2012Metric, F.Cu at (156.2, 78.8)
- added C35: 22uF, Capacitor_SMD:C_0805_2012Metric, F.Cu at (156.2, 80.8)
- added C36: 22uF, Capacitor_SMD:C_0805_2012Metric, F.Cu at (156.2, 82.8)
- added C37: 22uF, Capacitor_SMD:C_0805_2012Metric, F.Cu at (152.8, 78.8)
- added C38: 22uF, Capacitor_SMD:C_0805_2012Metric, F.Cu at (152.8, 82.8)
- added C39: 22uF, Capacitor_SMD:C_0805_2012Metric, F.Cu at (152.8, 80.8)
- added C40: 1nF, Capacitor_SMD:C_0402_1005Metric, F.Cu at (186.8, 75.8)
- added C41: 1nF, Capacitor_SMD:C_0402_1005Metric, F.Cu at (169.8, 111.0)
- added C42: 1nF, Capacitor_SMD:C_0402_1005Metric, F.Cu at (186.8, 79.8)
- added C43: 22uF, Capacitor_SMD:C_0805_2012Metric, F.Cu at (129.2, 109.0)
- added C44: 22uF, Capacitor_SMD:C_0805_2012Metric, F.Cu at (136.8, 109.5)
- added C45: 1nF, Capacitor_SMD:C_0402_1005Metric, F.Cu at (190.9, 80.5)
- added C46: 0.1uF, Capacitor_SMD:C_0402_1005Metric, F.Cu at (191.2, 84.8)
- added C47: 0.1uF, Capacitor_SMD:C_0402_1005Metric, F.Cu at (192.2, 89.8)
- added C48: 0.1uF, Capacitor_SMD:C_0402_1005Metric, F.Cu at (194.8, 94.5)
- added C49: 0.1uF, Capacitor_SMD:C_0402_1005Metric, F.Cu at (171.5, 75.5)
- added C50: 0.1uF, Capacitor_SMD:C_0402_1005Metric, F.Cu at (174.9, 80.6)
- added D3: BAT48ZFILM, Diode_SMD:D_SOD-123, F.Cu at (130.2, 99.8)
- added D4: SMAJ30A, Diode_SMD:D_SMA, F.Cu at (164.8, 102.0)
- added D5: Orange, LED_SMD:LED_0603_1608Metric, F.Cu at (170.0, 108.0)
- added J4: ~, xt30:XT30(2+2)PB-M.G.B, F.Cu at (130.0, 98.0)
- added J5: ~, xt30:XT30(2+2)PB-M.G.B, F.Cu at (170.0, 101.8)
- added Q2: TSM6502CR RLG, fet:TRANS_TSM6502CR_RLG, F.Cu at (150.4, 120.4)
- added Q3: TSM6502CR RLG, fet:TRANS_TSM6502CR_RLG, F.Cu at (164.7, 114.0)
- added Q4: TSM6502CR RLG, fet:TRANS_TSM6502CR_RLG, F.Cu at (164.7, 86.8)
- added Q5: BSS138, Package_TO_SOT_SMD:SOT-23, F.Cu at (161.0, 81.8)
- added Q6: BSS138, Package_TO_SOT_SMD:SOT-23, F.Cu at (156.5, 119.5)
- added Q7: BSS138, Package_TO_SOT_SMD:SOT-23, F.Cu at (160.4, 117.5)
- added R13: 0.02, Resistor_SMD:R_0805_2012Metric, F.Cu at (198.2, 82.8)
- added R14: 1.5k, Resistor_SMD:R_0402_1005Metric, F.Cu at (201.3, 86.8)
- added R17: 1.5k, Resistor_SMD:R_0402_1005Metric, F.Cu at (195.5, 88.2)
- added R18: 2k, Resistor_SMD:R_0402_1005Metric, F.Cu at (201.3, 91.8)
- added R19: 2k, Resistor_SMD:R_0402_1005Metric, F.Cu at (206.8, 72.5)
- added R20: 1.5k, Resistor_SMD:R_0402_1005Metric, F.Cu at (205.3, 81.8)
- added R23: 10, Resistor_SMD:R_0603_1608Metric, F.Cu at (211.0, 88.0)
- added R24: 1.5k, Resistor_SMD:R_0402_1005Metric, F.Cu at (209.5, 83.2)
- added R25: 10k, Resistor_SMD:R_0402_1005Metric, F.Cu at (205.3, 89.3)
- added R26: 10, Resistor_SMD:R_0805_2012Metric, F.Cu at (133.8, 105.2)
- added R27: 2k, Resistor_SMD:R_0402_1005Metric, F.Cu at (209.5, 93.0)
- added R28: 1.5k, Resistor_SMD:R_0402_1005Metric, F.Cu at (212.0, 73.0)
- added R29: 10, Resistor_SMD:R_0603_1608Metric, F.Cu at (214.5, 78.0)
- added R3: 10, Resistor_SMD:R_0603_1608Metric, F.Cu at (198.2, 74.5)
- added R30: 1.5k, Resistor_SMD:R_0402_1005Metric, F.Cu at (210.0, 77.8)
- added R31: 10k, Resistor_SMD:R_0402_1005Metric, F.Cu at (214.8, 84.5)
- added R32: 1k, Resistor_SMD:R_0402_1005Metric, F.Cu at (192.2, 102.0)
- added R4: 10k, Resistor_SMD:R_0402_1005Metric, F.Cu at (202.5, 72.8)
- added U6: INA180B2, Package_TO_SOT_SMD:SOT-23-5, F.Cu at (164.5, 96.0)
- added U7: M2003FC1AE, Package_SO:TSSOP-20_4.4x6.5mm_P0.65mm, F.Cu at (140.0, 115.5)
- added U8: MC78L05_SOT89, Package_TO_SOT_SMD:SOT-89-3, F.Cu at (133.0, 109.2)
- C1: value 10nF -> 470uF; footprint Capacitor_SMD:C_0402_1005Metric -> Capacitor_THT:C_Radial_D8.0mm_H7.0mm_P3.50mm
- C2: value 1uF -> 470uF; footprint Capacitor_SMD:C_0402_1005Metric -> Capacitor_THT:C_Radial_D8.0mm_H7.0mm_P3.50mm
- J2: value ~ -> Conn_01x05_Pin; footprint xt30:XT30(2+2)PB-M.G.B -> Connector_PinHeader_2.54mm:PinHeader_1x05_P2.54mm_Vertical
- R1: value 5.1k -> 0; footprint Resistor_SMD:R_0402_1005Metric -> Resistor_SMD:R_0603_1608Metric
- R15: value 470k -> 1.5k
- R2: value 22 -> 0; footprint Resistor_SMD:R_0402_1005Metric -> Resistor_SMD:R_0603_1608Metric
- R5: value 1k -> 0; footprint Resistor_SMD:R_0402_1005Metric -> Resistor_SMD:R_0603_1608Metric
- R6: value 1k -> 10k
- U1: value DRV8316RRGFR -> DRV5013; footprint DRV8316:drv -> Package_TO_SOT_SMD:SOT-23; moved to B.Cu
- U2: value RP2350A -> DRV5013; footprint MCU:RP2350-QFN-60-1EP_7x7_P0.4mm_EP3.4x3.4mm_ThermalVias -> Package_TO_SOT_SMD:SOT-23; moved to B.Cu
- U3: value W25Q128JVPIQ -> DRV5013; footprint Package_SON:WSON-8-1EP_6x5mm_P1.27mm_EP3.4x4.3mm -> Package_TO_SOT_SMD:SOT-23; moved to B.Cu
- U4: value MCP2518FD-xQBB -> LTC2850xDD; footprint Package_DFN_QFN:DFN-14-1EP_3x4.5mm_P0.65mm_EP1.65x4.25mm -> Package_DFN_QFN:DFN-8-1EP_3x3mm_P0.5mm_EP1.66x2.38mm
- moved R5 87.9 mm to (188.3, 109.5)
- moved R6 71.6 mm to (175.0, 71.5)
- moved U4 51.5 mm to (131.8, 89.8)
- moved R15 33.9 mm to (180.5, 76.0)
- moved U3 33.1 mm to (150.0, 122.2), turned to 180 degrees
- moved U2 32.9 mm to (141.0, 120.3), turned to 156 degrees
- moved R2 27.1 mm to (169.8, 109.8)
- moved C2 26.2 mm to (136.0, 86.2)
- moved C1 20.9 mm to (143.8, 82.2)
- moved R1 20.5 mm to (187.5, 95.5)
- moved J2 18.5 mm to (143.5, 73.7)
- moved U1 7.95 mm to (133.5, 114.8), turned to 132 degrees
Connections:
- C1 pad 1: Net-(U1-CPL) -> VBUS
- C1 pad 2: Net-(U1-CPH) -> GND
- C2 pad 2: Net-(U1-CP) -> GND
- J2 pad 1: unconnected-(J2-Pad1) -> +5V
- J2 pad 2: unconnected-(J2-Pad2) -> SSI_CSN
- R1 pad 1: +3V3 -> U
- R1 pad 2: /Motor Drive/nFAULT -> Net-(C40-Pad1)
- R15 pad 1: VBUS -> GND
- R15 pad 2: Net-(Q1-D) -> VDET
- R2 pad 1: Net-(U1-SW_BK) -> V
- R2 pad 2: Net-(U1-FB_BK) -> Net-(C41-Pad1)
- R5 pad 1: /microcontroller/LED0 -> W
- R6 pad 1: /microcontroller/LED1 -> VDET
- R6 pad 2: Net-(D2-A) -> VBUS
- U1 pad 1: unconnected-(U1-NC-Pad1) -> +5V
- U1 pad 2: GND -> HALL_A
- U1 pad 3: Net-(U1-FB_BK) -> GND
- U2 pad 1: +3V3 -> +5V
- U2 pad 2: unconnected-(U2-GPIO0-Pad2) -> HALL_B
- U2 pad 3: unconnected-(U2-GPIO1-Pad3) -> GND
- U3 pad 1: /microcontroller/QSPI_CS -> +5V
- U3 pad 2: /microcontroller/QSPI_IO1 -> HALL_C
- U3 pad 3: /microcontroller/QSPI_IO2 -> GND
- U4 pad 1: unconnected-(U4-TXCAN-Pad1) -> SWCLK
- U4 pad 2: unconnected-(U4-RXCAN-Pad2) -> DE
- U4 pad 3: unconnected-(U4-CLKO/SOF-Pad3) -> DE
- U4 pad 4: unconnected-(U4-~{INT}-Pad4) -> SWDIO
- U4 pad 5: unconnected-(U4-OSC2-Pad5) -> GND
- U4 pad 6: unconnected-(U4-OSC1-Pad6) -> Net-(U4-A)
- U4 pad 7: Net-(U4-VSS-Pad15) -> Net-(U4-B)
- U4 pad 8: unconnected-(U4-~{INT1}/GPIO1-Pad8) -> +5V
- U4 pad 9: unconnected-(U4-~{INT0}/GPIO0/XSTBY-Pad9) -> GND
Other:
- outline, holes or cut-outs redrawn
