File: drive.kicad_pcb (KiCad board)
At the start: 2 copper layers, 48 x 48 mm, 66 parts, among them J2 Conn_01x05_Pin, Q2 TSM6502CR RLG, Q3 TSM6502CR RLG, Q4 TSM6502CR RLG, Q5 BSS138, Q6 BSS138, Q7 BSS138, U1 DRV5013, U2 DRV5013, U3 DRV5013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

Commit message: pcb progress
Parts:
- removed C2: 470uF, Capacitor_THT:C_Radial_D8.0mm_H7.0mm_P3.50mm
- removed C38, C39: 22uF, Capacitor_SMD:C_0805_2012Metric
- added J1: Conn_ARM_JTAG_SWD_10, kuleana:SAMTEC_FTSH-105-XX-X-DV, F.Cu at (138.0, 86.5)
