File: drive.kicad_sch (KiCad schematic)
At the start: 0 parts

Commit message: m2003 drive
Parts:
- added C19, C30, C31: 1nF, symbol Device:C_Small
- added C32, C33: 0.1uF, symbol Device:C_Small
- added Q2, Q3, Q4: TSM6502CR RLG, fet:TRANS_TSM6502CR_RLG, symbol g431_esc:TSM6502CR
- added Q5, Q6, Q7: BSS138, Package_TO_SOT_SMD:SOT-23, symbol Transistor_FET:BSS138
- added R13: 0.01, Resistor_SMD:R_0603_1608Metric, symbol Device:R_Small
- added R14, R17, R20, R24, R28, R30: 1.5k, Resistor_SMD:R_0603_1608Metric, symbol Device:R_Small
- added R18, R19, R27: 2k, Resistor_SMD:R_0603_1608Metric, symbol Device:R_Small
- added R23, R29, R3: 10, Resistor_SMD:R_0603_1608Metric, symbol Device:R_Small
- added R25, R31, R4: 10k, Resistor_SMD:R_0603_1608Metric, symbol Device:R_Small
- added U6: INA180B2, Package_TO_SOT_SMD:SOT-23-5, symbol Amplifier_Current:INA180B2
- added U7: M2003FC1AE, Package_SO:TSSOP-20_4.4x6.5mm_P0.65mm, symbol MCU:M2003FC1AE
Connections:
- new net: C30.2, Q3.4 (G2), R20.2, R24.1
- new net: Q2.2 (G1), R3.2, R4.2
- new net: C31.2, Q4.4 (G2), R28.2, R30.1
- new net: Q5.3 (D), R14.1
- new net: C19.2, Q2.4 (G2), R14.2, R17.1
- new net: Q7.3 (D), R28.1
- new net: Q3.2 (G1), R23.2, R25.2
- new net: Q2.1 (S1), Q3.1 (S1), Q4.1 (S1), R13.2, U6.1 (+)
- new net: Q4.2 (G1), R29.2, R31.2
- new net: Q6.3 (D), R20.1
- new net +5V: C32.1, C33.2, U6.5 (V+), U7.9 (VDD)
- new net CS: U6.4, U7.2 (PB.2)
- new net GND: C32.2, C33.1, Q5.2 (S), Q6.2 (S), Q7.2 (S), R13.1, R18.1, R19.1, R25.1, R27.1, R31.1, R4.1, U6.2 (GND), U6.3 (-), U7.7 (VSS)
- new net HA: U7.10 (PC.14)
- new net HB: U7.6 (PB.5)
- new net HC: U7.5 (PB.4)
- new net RESET: U7.4 (PE.15/Reset)
- new net SSI_CSN: U7.1 (PB.1)
- new net SWCLK: U7.18 (PF.1/ICE_CLK)
- new net SWDIO: U7.8 (PF.0/ICE_DAT)
- new net U: Q2.5_6 (D2), Q2.7_8 (D1)
- new net UB: R3.1, U7.13 (PB.13)
- new net UT: Q5.1 (G), R18.2, U7.14 (PB.12)
- new net V: Q3.5_6 (D2), Q3.7_8 (D1)
- new net VB: R23.1, U7.16 (PB.8)
- new net VBUS: C19.1, C30.1, C31.1, Q2.3 (S2), Q3.3 (S2), Q4.3 (S2), R17.2, R24.2, R30.2
- new net VT: Q6.1 (G), R19.2, U7.15 (PB.7)
- new net W: Q4.5_6 (D2), Q4.7_8 (D1)
- new net WB: R29.1, U7.17 (PB.9)
- new net WT: Q7.1 (G), R27.2, U7.19 (PB.11)
Other:
- sheet Motor Drive ports: added CS, CSA, CSB, CSC, DRV_OFF, INHA, INHB, INHC, INLA, INLB, INLC, MISO, MOSI, SCK, VREF/ILIM, nFAULT; removed none
- sheet microcontroller ports: added DRV_CS, DRV_CSA, DRV_CSB, DRV_CSC, DRV_FAULT, DRV_OFF, INHA, INHB, INHC, INLA, INLB, INLC, MISO, MOSI, SCK, VREF/ILIM; removed none

Commit message: schematic complete
Parts:
- added C1, C2: 470uF, Capacitor_THT:C_Radial_D8.0mm_H7.0mm_P3.50mm, symbol Device:C_Small_US
- added C34, C35, C36, C37, C38, C39, C43, C44: 22uF, Capacitor_SMD:C_0805_2012Metric, symbol Device:C_Small
- added C40, C41, C42, C45: 1nF, Capacitor_SMD:C_0402_1005Metric, symbol Device:C_Small
- added C46, C47, C48, C49, C50: 0.1uF, Capacitor_SMD:C_0402_1005Metric, symbol Device:C_Small
- added D3: BAT48ZFILM, Diode_SMD:D_SOD-123, symbol Diode:BAT48ZFILM
- added D4: SMAJ30A, Diode_SMD:D_SMA, symbol Diode:SMAJ30A
- added D5: Orange, LED_SMD:LED_0603_1608Metric, symbol kuleana:LED
- added J1: Conn_ARM_JTAG_SWD_10, kuleana:SAMTEC_FTSH-105-XX-X-DV, symbol Connector:Conn_ARM_JTAG_SWD_10
- added J2: Conn_01x05_Pin, Connector_PinHeader_2.54mm:PinHeader_1x05_P2.54mm_Vertical, symbol Connector:Conn_01x05_Pin
- added J4, J5: (no value), xt30:XT30(2+2)PB-M.G.B, symbol MSconnector:XT30(2+2)
- added R1, R2, R5: 0, Resistor_SMD:R_0603_1608Metric, symbol Device:R_Small
- added R15: 1.5k, Resistor_SMD:R_0402_1005Metric, symbol Device:R_Small
- added R26: 10, Resistor_SMD:R_0805_2012Metric, symbol Device:R_Small
- added R32: 1k, Resistor_SMD:R_0402_1005Metric, symbol kuleana:R
- added R6: 10k, Resistor_SMD:R_0402_1005Metric, symbol Device:R_Small
- added U1, U2, U3: DRV5013, Package_TO_SOT_SMD:SOT-23, symbol Sensor_Magnetic:DRV5033FAxDBZ
- added U4: LTC2850xDD, Package_DFN_QFN:DFN-8-1EP_3x3mm_P0.5mm_EP1.66x2.38mm, symbol Interface_UART:LTC2850xDD
- added U8: MC78L05_SOT89, Package_TO_SOT_SMD:SOT-89-3, symbol Regulator_Linear:MC78L05_SOT89
- C19, C30, C31, C32, C33: footprint (none) -> Capacitor_SMD:C_0402_1005Metric
- R13: value 0.01 -> 0.02; footprint Resistor_SMD:R_0603_1608Metric -> Resistor_SMD:R_0805_2012Metric
- R14, R17, R18, R19, R20, R24, R25, R27, R28, R30, R31, R4: footprint Resistor_SMD:R_0603_1608Metric -> Resistor_SMD:R_0402_1005Metric
Connections:
- net +5V: now also C44.1, C46.2, C47.2, C48.2, C50.2, J1.1 (VTref), J2.1 (Pin_1), U1.1 (VCC), U2.1 (VCC), U3.1 (VCC), U4.8 (VCC), U8.1 (OUT)
- net GND: now also C1.2, C2.2, C34.2, C35.2, C36.2, C37.2, C38.2, C39.2, C40.2, C41.2, C42.2, C43.2, C44.2, C45.2, C46.1, C47.1, C48.1, C49.1, C50.1, D4.2 (A2), D5.1 (K), J1.3 (GND), J1.5 (GND), J1.9 (GNDDetect), J2.5 (Pin_5), J4.-, J5.-, R15.1, U1.3 (GND), U2.3 (GND), U3.3 (GND), U4.5 (GND), U4.9 (GND), U8.2 (GND)
- net RESET: now also J1.10 (~{RESET})
- net SSI_CLK: now also U7.20 (PB.0), J2.3 (Pin_3)
- net SSI_CSN: now also J2.2 (Pin_2), R32.1
- net SSI_DAT: now also U7.11 (PB.15), J2.4 (Pin_4)
- net SWCLK: now also J1.4 (SWCLK/TCK), U4.1 (RO)
- net SWDIO: now also J1.2 (SWDIO/TMS), U4.4 (DI)
- net U: now also R1.1
- net V: now also R2.1
- net VBUS: now also C1.1, C2.1, C34.1, C35.1, C36.1, C37.1, C38.1, C39.1, C45.1, D3.2 (A), D4.1 (A1), J4.+, J5.+, R6.2
- net W: now also R5.1
- net DE: now reaches U7.12 (PB.14)
- net DE: now also U4.2 (~{RE}), U4.3 (DE)
- net VDET: now reaches U7.3 (PB.3)
- net VDET: now also C49.2, R15.2, R6.1
- net HA renamed HALL_A
- net HALL_A: now also U1.2 (OUT)
- net HB renamed HALL_B
- net HALL_B: now also U2.2 (OUT)
- net HC renamed HALL_C
- net HALL_C: now also U3.2 (OUT)
- new net: J4.1, J5.1, U4.6 (A)
- new net: J4.2, J5.2, U4.7 (B)
- new net: C40.1, R1.2
- new net: C42.1, R5.2
- new net: D5.2 (A), R32.2
- new net: D3.1 (K), R26.1
- new net: C43.1, R26.2, U8.3 (IN)
- new net: C41.1, R2.2
- no-connect marks 0 -> 2
Other:
- removed sheet CAN
- removed sheet Motor Drive
- removed sheet microcontroller
- removed sheet power
- moved on the sheet: C19, C30, C31, C32, C33, Q2A, Q2B, Q3A, Q3B, Q4A, Q4B, Q5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
