File: drive.kicad_sch (KiCad schematic)
At the start: 67 parts, among them J1 Conn_ARM_JTAG_SWD_10, J2 Conn_01x05_Pin, Q2 TSM6502CR RLG, Q3 TSM6502CR RLG, Q4 TSM6502CR RLG, Q5 BSS138, Q6 BSS138, Q7 BSS138, U1 DRV5013, U2 DRV5013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

Commit message: pcb progress
Parts:
- removed C2: 470uF, Capacitor_THT:C_Radial_D8.0mm_H7.0mm_P3.50mm, symbol Device:C_Small_US
- removed C38, C39: 22uF, Capacitor_SMD:C_0805_2012Metric, symbol Device:C_Small
Other:
- moved on the sheet: C1
